File: day1-power-board/day1-power-board.kicad_pcb (KiCad board)
At the start: 2 copper layers, 69 x 31 mm, 10 parts, among them J1 V_IN, J2 V_OUT, U1 L78L05_SOT89

Commit message: Add 5V test point
Parts:
- added TP1: 5V_TEST, TestPoint:TestPoint_Pad_2.0x2.0mm, F.Cu at (168.5, 80.5)
Routing:
- net +5V: track 36.7 -> 45.3 mm
Changed lines of the file:
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@@
 		)
+	)
+	(footprint "TestPoint:TestPoint_Pad_2.0x2.0mm"
+		(layer "F.Cu")
+		(at 168.5 80.5)
+		(descr "SMD rectangular pad as test Point, square 2.0mm side length")
+		(tags "test point SMD pad rectangle square")
+		(property "Reference" "TP1"
+			(at 0 -1.998 0)
+			(layer "F.SilkS")
+			(effects
+				(font
+					(size 1 1)
+					(thickness 0.15)
+				)
+			)
+		)
+		(property "Value" "5V_TEST"
+			(at 0 2.05 0)
+			(layer "F.Fab")
+			(effects
+				(font
+					(size 1 1)
+					(thickness 0.15)
+				)
+			)
+		)
+		(property "Datasheet" "~"
+			(at 0 0 0)
+			(unlocked yes)
+			(layer "F.Fab")
+			(hide yes)
+			(effects
+				(font
+					(size 1.27 1.27)
+					(thickness 0.15)
+				)
+			)
+		)
+		(property "Description" "test point"
+			(at 0 0 0)
+			(unlocked yes)
+			(layer "F.Fab")
+			(hide yes)
+			(effects
+				(font
+					(size 1.27 1.27)
+					(thickness 0.15)
+				)
+			)
+		)
+		(property ki_fp_filters "Pin* Test*")
+		(sheetname "/")
+		(sheetfile "day1-power-board.kicad_sch")
+		(attr exclude_from_pos_files)
+		(fp_line
+			(start -1.2 -1.2)
+			(end 1.2 -1.2)
+			(stroke
+				(width 0.12)
+				(type solid)
+			)
+			(layer "F.SilkS")
+		)
+		(fp_line
+			(start -1.2 1.2)
+			(end -1.2 -1.2)
+			(stroke
+				(width 0.12)
+				(type solid)
+			)
+			(layer "F.SilkS")
+		)
+		(fp_line
+			(start 1.2 -1.2)
+			(end 1.2 1.2)
+			(stroke
+				(width 0.12)
+				(type solid)
+			)
+			(layer "F.SilkS")
+		)
+		(fp_line
+			(start 1.2 1.2)
+			(end -1.2 1.2)
+			(stroke
+				(width 0.12)
+				(type solid)
+			)
+			(layer "F.SilkS")
+		)
+		(fp_line
+			(start -1.5 -1.5)
+			(end -1.5 1.5)
+			(stroke
+				(width 0.05)
+				(type solid)
+			)
+			(layer "F.CrtYd")
+		)
+		(fp_line
+			(start -1.5 -1.5)
+			(end 1.5 -1.5)
+			(stroke
+				(width 0.05)
+				(type solid)
+			)
+			(layer "F.CrtYd")
+		)
+		(fp_line
+			(start 1.5 1.5)
+			(end -1.5 1.5)
+			(stroke
+				(width 0.05)
+				(type solid)
+			)
+			(layer "F.CrtYd")
+		)
+		(fp_line
+			(start 1.5 1.5)
+			(end 1.5 -1.5)
+			(stroke
+				(width 0.05)
+				(type solid)
+			)
+			(layer "F.CrtYd")
+		)
+		(fp_text user "${REFERENCE}"
+			(at 0 -2 0)
+			(layer "F.Fab")
+			(effects
+				(font
+					(size 1 1)
+					(thickness 0.15)
+				)
+			)
+		)
+		(pad "1" smd rect
+			(at 0 0)
+			(size 2 2)
+			(layers "F.Cu" "F.Mask")
+			(net 3 "+5V")
+			(pinfunction "1")
+			(pintype "passive")
+		)
+		(embedded_fonts no)
 	)
 	(footprint "Capacitor_SMD:C_0805_2012Metric"
@@
 	)
 	(segment
+		(start 165.5 83.5)
+		(end 168.5 80.5)
+		(width 0.5)
+		(layer "F.Cu")
+		(net 3)
+	)
+	(segment
 		(start 148.5 91.5)
 		(end 152.5 91.5)
@@
 		(width 0.5)
 		(layer "F.Cu")
+		(net 3)
+	)
+	(segment
+		(start 165.5 87.8275)
+		(end 165.5 83.5)
+		(width 0.5)
+		(layer "F.Cu")

Commit message: Add custom sensor footprint
Parts:
- added U2: RPR-0521RS, MYLIBRARY:MY_SENSOR_1x04_P2.54mm, F.Cu at (126.4, 117.0)
Changed lines of the file:
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@@
 	(net 4 "/12V_RAW")
 	(net 5 "Net-(D2-K)")
+	(net 6 "unconnected-(U2-VDD-Pad1)")
+	(net 7 "unconnected-(U2-GND-Pad3)")
+	(net 8 "unconnected-(U2-LED_A-Pad4)")
+	(net 9 "unconnected-(U2-SCL-Pad2)")
 	(footprint "Resistor_SMD:R_0805_2012Metric"
 		(layer "F.Cu")
@@
 		)
 	)
+	(footprint "MYLIBRARY:MY_SENSOR_1x04_P2.54mm"
+		(layer "F.Cu")
+		(at 126.38 117)
+		(property "Reference" "U2"
+			(at 0 -6.5 0)
+			(unlocked yes)
+			(layer "F.SilkS")
+			(effects
+				(font
+					(size 1 1)
+					(thickness 0.1)
+				)
+			)
+		)
+		(property "Value" "RPR-0521RS"
+			(at 0 7.5 0)
+			(unlocked yes)
+			(layer "F.Fab")
+			(effects
+				(font
+					(size 1 1)
+					(thickness 0.15)
+				)
+			)
+		)
+		(property "Datasheet" "https://fscdn.rohm.com/en/products/databook/datasheet/opto/optical_sensor/opto_module/rpr-0521rs-e.pdf"
+			(at 0 0 0)
+			(unlocked yes)
+			(layer "F.Fab")
+			(hide yes)
+			(effects
+				(font
+					(size 1 1)
+					(thickness 0.15)
+				)
+			)
+		)
+		(property "Description" "Digital Proximity and Ambient Light Sensor"
+			(at 0 0 0)
+			(unlocked yes)
+			(layer "F.Fab")
+			(hide yes)
+			(effects
+				(font
+					(size 1 1)
+					(thickness 0.15)
+				)
+			)
+		)
+		(property ki_fp_filters "Rohm?RPR?0521*")
+		(sheetname "/")
+		(sheetfile "day1-power-board.kicad_sch")
+		(attr smd)
+		(fp_line
+			(start -1.5 -1)
+			(end -1.5 1.5)
+			(stroke
+				(width 0.1)
+				(type dot)
+			)
+			(layer "F.SilkS")
+		)
+		(fp_line
+			(start -1.5 1.5)
+			(end -0.5 1.5)
+			(stroke
+				(width 0.1)
+				(type dot)
+			)
+			(layer "F.SilkS")
+		)
+		(fp_rect
+			(start -3.5 -4)
+			(end 10.5 3.5)
+			(stroke
+				(width 0.05)
+				(type default)
+			)
+			(fill no)
+			(layer "Edge.Cuts")
+		)
+		(fp_rect
+			(start -4.5 -4.5)
+			(end 11.5 4)
+			(stroke
+				(width 0.05)
+				(type default)
+			)
+			(fill no)
+			(layer "F.CrtYd")
+		)
+		(fp_text user "${REFERENCE}"
+			(at 0 9 0)
+			(unlocked yes)
+			(layer "F.Fab")
+			(effects
+				(font
+					(size 1 1)
+					(thickness 0.15)
+				)
+			)
+		)
+		(pad "1" smd roundrect
+			(at 0 0)
+			(size 1.905 1.27)
+			(layers "F.Cu" "F.Mask" "F.Paste")
+			(roundrect_rratio 0.15)
+			(net 6 "unconnected-(U2-VDD-Pad1)")
+			(pinfunction "VDD")
+			(pintype "power_in")
+		)
+		(pad "2" smd roundrect
+			(at 2.54 0)
+			(size 1.905 1.27)
+			(layers "F.Cu" "F.Mask" "F.Paste")
+			(roundrect_rratio 0.15)
+			(net 9 "unconnected-(U2-SCL-Pad2)")
+			(pinfunction "SCL")
+			(pintype "input")
+		)
+		(pad "3" smd roundrect
+			(at 5.08 0)
+			(size 1.905 1.27)
+			(layers "F.Cu" "F.Mask" "F.Paste")
+			(roundrect_rratio 0.15)
+			(net 7 "unconnected-(U2-GND-Pad3)")
+			(pinfunction "GND")
+			(pintype "power_in")
+		)
+		(pad "4" smd roundrect
+			(at 7.62 0)
+			(size 1.905 1.27)
+			(layers "F.Cu" "F.Mask" "F.Paste")
+			(roundrect_rratio 0.15)
+			(net 8 "unconnected-(U2-LED_A-Pad4)")
+			(pinfunction "LED_A")
+			(pintype "passive")
+		)
+		(embedded_fonts no)
+	)
 	(footprint "Package_TO_SOT_THT:TO-220-3_Vertical"
