File: day1-power-board/power.kicad_sch (KiCad schematic)
At the start: 11 parts, among them J1 V_IN, J2 V_OUT, U1 L78L05_SOT89

Commit message: Clean up hierarchical schematic
Connections:
- net +5V renamed 5V_OUT
Changed lines of the file:
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@@
 	(wire
 		(pts
-			(xy 198.12 73.66) (xy 198.12 74.93)
+			(xy 198.12 68.58) (xy 198.12 74.93)
 		)
 		(stroke
@@
 	(wire
 		(pts
-			(xy 204.47 73.66) (xy 198.12 73.66)
-		)
-		(stroke
-			(width 0)
-			(type default)
-		)
-	)
-	(wire
-		(pts
 			(xy 198.12 74.93) (xy 194.31 74.93)
 		)
@@
 		(pts
 			(xy 102.87 102.87) (xy 118.11 102.87)
-		)
-		(stroke
-			(width 0)
-			(type default)
-		)
-	)
-	(wire
-		(pts
-			(xy 194.31 73.66) (xy 194.31 74.93)
 		)
 		(stroke
@@
 	(hierarchical_label "5V_OUT"
 		(shape input)
-		(at 204.47 73.66 0)
+		(at 198.12 68.58 0)
 		(effects
 			(font
@@
 					(unit 1)
 				)
-			)
-		)
-	)
-	(symbol
-		(lib_id "power:+5V")
-		(at 194.31 73.66 0)
-		(unit 1)
-		(exclude_from_sim no)
-		(in_bom yes)
-		(on_board yes)
-		(dnp no)
-		(fields_autoplaced yes)
-		(property "Reference" "#PWR05"
-			(at 194.31 77.47 0)
-			(effects
-				(font
-					(size 1.27 1.27)
-				)
-				(hide yes)
-			)
-		)
-		(property "Value" "+5V"
-			(at 194.31 68.58 0)
-			(effects
-				(font
-					(size 1.27 1.27)
-				)
-			)
-		)
-		(property "Footprint" ""
-			(at 194.31 73.66 0)
-			(effects
-				(font
-					(size 1.27 1.27)
-				)
-				(hide yes)
-			)
-		)
-		(property "Datasheet" ""
-			(at 194.31 73.66 0)
-			(effects
-				(font
-					(size 1.27 1.27)
-				)
-				(hide yes)
-			)
-		)
-		(property "Description" "Power symbol creates a global label with name \"+5V\""
-			(at 194.31 73.66 0)
-			(effects
-				(font
-					(size 1.27 1.27)
-				)
-				(hide yes)
-			)
-		)
-		(pin "1"
-		)
-		(instances
-			(project "day1-power-board"
-				(path "/36a2fab3-956e-472e-853f-9772f700f857/1ea3b6f2-161e-4151-b76b-a485480dee21"
-					(reference "#PWR05")
-					(unit 1)
-				)
